File: LMH6629_test.sch (EAGLE design)
At the start: 18 parts, among them X1 1-227161-0, X2 SMA-142-0711-871/876

Commit message: replace LDO on pcb
Parts:
- removed X2: SMA-142-0711-871/876, con-coax:SMA-142-0711-871/876
- added J1: (no value), con-jack:JACK-PLUG1
- added R6, R7: (no value), resistor:R-EU_R0603
- added X3: SMA-142-0701-801/806, con-coax:SMA-142-0701-801/806
Connections:
- removed net IN: C10.2, X2.1
- removed net V_OUT: U$1.OUT, X1.1
- new net N$1: R6.1, R7.2, U$1.OUT
- new net N$2: R6.2, X1.1
- new net N$3: C10.2, X3.1
- net GND: now also J1.1, J1.2, R7.1, X3.2; no longer X2.2
- net PWR_IN: now also J1.3
Other:
- moved on the sheet: X1
Changed lines of the file:
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@@
 <setting verticaltext="up"/>
 </settings>
-<grid distance="0.1" unitdist="inch" unit="inch" style="lines" multiple="1" display="yes" altdistance="0.01" altunitdist="inch" altunit="inch"/>
+<grid distance="0.1" unitdist="inch" unit="inch" style="lines" multiple="1" display="no" altdistance="0.01" altunitdist="inch" altunit="inch"/>
 <layers>
 <layer number="1" name="Top" color="4" fill="1" visible="no" active="no"/>
@@
 <layer number="51" name="tDocu" color="7" fill="1" visible="no" active="no"/>
 <layer number="52" name="bDocu" color="7" fill="1" visible="no" active="no"/>
+<layer number="53" name="tGND_GNDA" color="7" fill="9" visible="no" active="no"/>
+<layer number="54" name="bGND_GNDA" color="1" fill="9" visible="no" active="no"/>
 <layer number="56" name="wert" color="7" fill="1" visible="no" active="no"/>
 <layer number="90" name="Modules" color="5" fill="1" visible="yes" active="yes"/>
@@
 <layer number="98" name="Guide" color="6" fill="1" visible="yes" active="yes"/>
 <layer number="99" name="SpiceOrder" color="5" fill="1" visible="yes" active="yes"/>
+<layer number="100" name="Muster" color="7" fill="1" visible="no" active="no"/>
+<layer number="102" name="Vscore" color="7" fill="1" visible="no" active="yes"/>
+<layer number="104" name="Name" color="7" fill="1" visible="no" active="yes"/>
+<layer number="151" name="HeatSink" color="14" fill="1" visible="no" active="no"/>
+<layer number="200" name="200bmp" color="1" fill="10" visible="no" active="no"/>
+<layer number="201" name="201bmp" color="2" fill="1" visible="no" active="no"/>
+<layer number="202" name="202bmp" color="3" fill="1" visible="no" active="no"/>
+<layer number="203" name="203bmp" color="4" fill="10" visible="no" active="no"/>
+<layer number="204" name="204bmp" color="5" fill="10" visible="no" active="no"/>
+<layer number="205" name="205bmp" color="6" fill="10" visible="no" active="no"/>
+<layer number="206" name="206bmp" color="7" fill="10" visible="no" active="no"/>
+<layer number="207" name="207bmp" color="15" fill="10" visible="no" active="no"/>
+<layer number="217" name="217bmp" color="18" fill="1" visible="no" active="no"/>
+<layer number="218" name="218bmp" color="19" fill="1" visible="no" active="no"/>
+<layer number="219" name="219bmp" color="20" fill="1" visible="no" active="no"/>
+<layer number="220" name="220bmp" color="21" fill="1" visible="no" active="no"/>
+<layer number="221" name="221bmp" color="22" fill="1" visible="no" active="no"/>
+<layer number="222" name="222bmp" color="23" fill="1" visible="no" active="no"/>
+<layer number="223" name="223bmp" color="24" fill="1" visible="no" active="no"/>
+<layer number="224" name="224bmp" color="25" fill="1" visible="no" active="no"/>
+<layer number="250" name="Descript" color="3" fill="1" visible="no" active="no"/>
+<layer number="251" name="SMDround" color="12" fill="11" visible="no" active="no"/>
+<layer number="254" name="OrgLBR" color="13" fill="1" visible="no" active="no"/>
 </layers>
 <schematic xreflabel="%F%N/%S.%C%R" xrefpart="/%S.%C%R">
@@
 <part name="GND15" library="supply1" library_urn="urn:adsk.eagle:library:371" deviceset="GND" device=""/>
 <part name="C10" library="rcl" library_urn="urn:adsk.eagle:library:334" deviceset="C-EU" device="C0603" package3d_urn="urn:adsk.eagle:package:23616/2"/>
-<part name="X2" library="con-coax" library_urn="urn:adsk.eagle:library:133" deviceset="SMA-" device="142-0711-871/876" package3d_urn="urn:adsk.eagle:package:6217/1"/>
 <part name="GND16" library="supply1" library_urn="urn:adsk.eagle:library:371" deviceset="GND" device=""/>
 <part name="C11" library="rcl" library_urn="urn:adsk.eagle:library:334" deviceset="C-EU" device="C0603" package3d_urn="urn:adsk.eagle:package:23616/2"/>
 <part name="GND17" library="supply1" library_urn="urn:adsk.eagle:library:371" deviceset="GND" device=""/>
+<part name="R6" library="resistor" library_urn="urn:adsk.eagle:library:348" deviceset="R-EU_" device="R0603" package3d_urn="urn:adsk.eagle:package:26057/1"/>
+<part name="R7" library="resistor" library_urn="urn:adsk.eagle:library:348" deviceset="R-EU_" device="R0603" package3d_urn="urn:adsk.eagle:package:26057/1"/>
+<part name="GND10" library="supply1" library_urn="urn:adsk.eagle:library:371" deviceset="GND" device=""/>
+<part name="X3" library="con-coax" library_urn="urn:adsk.eagle:library:133" deviceset="SMA-" device="142-0701-801/806" package3d_urn="urn:adsk.eagle:package:6214/1"/>
+<part name="J1" library="con-jack" deviceset="JACK-PLUG" device="1"/>
+<part name="GND12" library="supply1" deviceset="GND" device=""/>
 </parts>
 <sheets>
@@
 <instance part="FRAME1" gate="G$1" x="0" y="0"/>
 <instance part="FRAME1" gate="G$2" x="162.56" y="0"/>
-<instance part="X1" gate="G$1" x="157.48" y="88.9" smashed="yes" rot="MR0">
-<attribute name="VALUE" x="167.64" y="83.82" size="1.778" layer="96" rot="MR0"/>
-<attribute name="NAME" x="160.02" y="92.202" size="1.778" layer="95" rot="MR0"/>
+<instance part="X1" gate="G$1" x="187.96" y="88.9" smashed="yes" rot="MR0">
+<attribute name="VALUE" x="198.12" y="83.82" size="1.778" layer="96" rot="MR0"/>
+<attribute name="NAME" x="190.5" y="92.202" size="1.778" layer="95" rot="MR0"/>
 </instance>
-<instance part="GND1" gate="1" x="152.4" y="81.28"/>
+<instance part="GND1" gate="1" x="182.88" y="81.28"/>
 <instance part="U$1" gate="G$1" x="106.68" y="81.28"/>
 <instance part="R1" gate="G$1" x="76.2" y="81.28" rot="R270"/>
@@
 <instance part="GND15" gate="1" x="55.88" y="139.7"/>
 <instance part="C10" gate="G$1" x="55.88" y="63.5" rot="R270"/>
-<instance part="X2" gate="G1" x="27.94" y="63.5"/>
 <instance part="GND16" gate="1" x="33.02" y="53.34"/>
 <instance part="C11" gate="G$1" x="144.78" y="109.22" rot="R180"/>
 <instance part="GND17" gate="1" x="144.78" y="119.38" rot="R180"/>
+<instance part="R6" gate="G$1" x="172.72" y="88.9"/>
+<instance part="R7" gate="G$1" x="160.02" y="81.28" rot="R90"/>
+<instance part="GND10" gate="1" x="160.02" y="71.12"/>
+<instance part="X3" gate="G1" x="27.94" y="63.5"/>
+<instance part="J1" gate="G$1" x="34.29" y="152.4"/>
+<instance part="GND12" gate="1" x="41.91" y="144.78"/>
 </instances>
 <busses>
@@
 <pinref part="X1" gate="G$1" pin="2"/>
 <pinref part="GND1" gate="1" pin="GND"/>
-<wire x1="154.94" y1="86.36" x2="152.4" y2="86.36" width="0.1524" layer="91"/>
-<wire x1="152.4" y1="86.36" x2="152.4" y2="83.82" width="0.1524" layer="91"/>
+<wire x1="185.42" y1="86.36" x2="182.88" y2="86.36" width="0.1524" layer="91"/>
+<wire x1="182.88" y1="86.36" x2="182.88" y2="83.82" width="0.1524" layer="91"/>
 </segment>
 <segment>
@@
 </segment>
 <segment>
-<pinref part="X2" gate="G1" pin="2"/>
+<pinref part="C11" gate="G$1" pin="2"/>
+<pinref part="GND17" gate="1" pin="GND"/>
+<wire x1="144.78" y1="114.3" x2="144.78" y2="116.84" width="0.1524" layer="91"/>
+</segment>
+<segment>
+<pinref part="R7" gate="G$1" pin="1"/>
+<pinref part="GND10" gate="1" pin="GND"/>
+<wire x1="160.02" y1="73.66" x2="160.02" y2="76.2" width="0.1524" layer="91"/>
+</segment>
+<segment>
+<pinref part="X3" gate="G1" pin="2"/>
 <pinref part="GND16" gate="1" pin="GND"/>
 <wire x1="30.48" y1="60.96" x2="33.02" y2="60.96" width="0.1524" layer="91"/>
@@
 </segment>
 <segment>
-<pinref part="C11" gate="G$1" pin="2"/>
-<pinref part="GND17" gate="1" pin="GND"/>
-<wire x1="144.78" y1="114.3" x2="144.78" y2="116.84" width="0.1524" layer="91"/>
-</segment>
-</net>
-<net name="V_OUT" class="0">
-<segment>
-<pinref part="U$1" gate="G$1" pin="OUT"/>
-<pinref part="X1" gate="G$1" pin="1"/>
-<wire x1="133.35" y1="88.9" x2="154.94" y2="88.9" width="0.1524" layer="91"/>
-<label x="142.24" y="88.9" size="1.778" layer="95"/>
+<pinref part="J1" gate="G$1" pin="2"/>
+<pinref part="GND12" gate="1" pin="GND"/>
+<wire x1="39.37" y1="152.4" x2="41.91" y2="152.4" width="0.1524" layer="91"/>
+<wire x1="41.91" y1="152.4" x2="41.91" y2="149.86" width="0.1524" layer="91"/>
+<pinref part="J1" gate="G$1" pin="1"/>
+<wire x1="41.91" y1="149.86" x2="41.91" y2="147.32" width="0.1524" layer="91"/>
+<wire x1="39.37" y1="149.86" x2="41.91" y2="149.86" width="0.1524" layer="91"/>
+<junction x="41.91" y="149.86"/>
 </segment>
 </net>
@@
 <pinref part="U$2" gate="G$1" pin="IN"/>
 <wire x1="86.36" y1="154.94" x2="88.9" y2="154.94" width="0.1524" layer="91"/>
-<wire x1="53.34" y1="154.94" x2="55.88" y2="154.94" width="0.1524" layer="91"/>
 <junction x="86.36" y="154.94"/>
 <pinref part="C4" gate="G$1" pin="1"/>
@@
 <pinref part="C8" gate="G$1" pin="1"/>
 <wire x1="55.88" y1="152.4" x2="55.88" y2="154.94" width="0.1524" layer="91"/>
+<label x="60.96" y="154.94" size="1.778" layer="95"/>
+<pinref part="J1" gate="G$1" pin="3"/>
+<wire x1="39.37" y1="154.94" x2="55.88" y2="154.94" width="0.1524" layer="91"/>
 <junction x="55.88" y="154.94"/>
-<label x="60.96" y="154.94" size="1.778" layer="95"/>
 </segment>
 </net>
@@
 </segment>
 </net>
-<net name="IN" class="0">
-<segment>
+<net name="N$1" class="0">
+<segment>
+<pinref part="U$1" gate="G$1" pin="OUT"/>
+<pinref part="R6" gate="G$1" pin="1"/>
+<wire x1="133.35" y1="88.9" x2="160.02" y2="88.9" width="0.1524" layer="91"/>
+<pinref part="R7" gate="G$1" pin="2"/>
+<wire x1="160.02" y1="88.9" x2="167.64" y2="88.9" width="0.1524" layer="91"/>
+<wire x1="160.02" y1="86.36" x2="160.02" y2="88.9" width="0.1524" layer="91"/>
+<junction x="160.02" y="88.9"/>
+</segment>
+</net>
+<net name="N$2" class="0">
+<segment>
+<pinref part="R6" gate="G$1" pin="2"/>
+<pinref part="X1" gate="G$1" pin="1"/>
+<wire x1="177.8" y1="88.9" x2="185.42" y2="88.9" width="0.1524" layer="91"/>
+</segment>
+</net>
+<net name="N$3" class="0">
+<segment>
+<pinref part="X3" gate="G1" pin="1"/>
 <pinref part="C10" gate="G$1" pin="2"/>
-<wire x1="50.8" y1="63.5" x2="30.48" y2="63.5" width="0.1524" layer="91"/>
-<label x="40.64" y="63.5" size="1.778" layer="95"/>
-<pinref part="X2" gate="G1" pin="1"/>
-</segment>
-</net>
+<wire x1="30.48" y1="63.5" x2="50.8" y2="63.5" width="0.1524" layer="91"/>
+</segment>
+</net>

Commit message: almost done with pcb
Parts:
- removed J1: (no value), con-jack:JACK-PLUG1
- added C5: (no value), rcl:C-EUC0603
- added LED1: (no value), adafruit:LEDCHIPLED_0603
- added R8: (no value), resistor:R-EU_R0603
- added X2: (no value), adafruit:SMACONNECTOR_EDGE
- R1, R2: device resistor:R-EU_R0603 -> resistor:R-EU_R0402
- R6, R7: value (none) -> 51R
- X3: value SMA-142-0701-801/806 -> (none); device con-coax:SMA-142-0701-801/806 -> con-jack:JACK-PLUG1
- renumbered U$1 to U1, U$2 to U2
Connections:
- net N$1 renamed V_OUT
- net N$2 renamed OUT
- net N$5 renamed -IN
- removed net N$6: R1.1, U1.FB
- new net FB: R2.2, U1.FB
- new net N$1: LED1.A, R8.1
- net GND: now also C5.2, LED1.C, R1.1, X2.GND1, X2.GND2, X2.GND3, X2.GND4, X3.1; no longer J1.1, J1.2, R2.2
- net N$3: now also X2.ANT; no longer X3.1
- net PWR_IN: now also X3.3; no longer J1.3
- net V_ANALOG: now also C5.1, R8.2
Other:
- moved on the sheet: C6, R1, R2

Commit message: all done
Parts:
- removed C2: (no value), rcl:C-EUC0805
- added C12: 22u, rcl:C-EUC0805
- added C13: 47u, resistor:C-EUC1210
- added C9: 51p, rcl:C-EUC0603
- C1: value (none) -> 0.01u
- C10: value (none) -> 1n
- C11, C4: value (none) -> 0.1u
- C3: value (none) -> 0.22u
- C5, C7: value (none) -> 1u
- C6: value (none) -> 4.7u
- C8: value (none) -> 10u
- R1, R8: value (none) -> 680R
- R2: value (none) -> 12R
- R3: value (none) -> 18k
- R4: value (none) -> 6.2k
- R5: value (none) -> 2.7k
- R7: value 51R -> 51R DNI
Connections:
- net -IN: now also R1.1, R2.2; no longer R1.2, R2.1
- net ADJ: now also C9.1
- net FB: now also R1.2; no longer R2.2
- net GND: now also C12.2, C13.2, R2.1; no longer C2.2, R1.1
- net PWR_IN: now also C13.1; no longer C2.1
- net V_ANALOG: now also C12.1, C9.2
Other:
- moved on the sheet: C3, C6, C8, R1, R2, R4
